Commit message: fix: Fixes the mimic tag problem by removing it. The result is that both joints are actuated which happens by deafult

File: robotiq_hande_description/urdf/robotiq_hande_gripper_processed.urdf (robot description, URDF)
Before this commit: robot robotiq_hande_gripper, 6 links, 5 joints
Joints:
- joint hande_right_finger_joint: mimic joint=hande_left_finger_joint multiplier=1 offset=0 -> (none)
